File: led_master.sch (EAGLE design)
At the start: 50 parts, among them IC2 MEGA8-AI, IC3 4081D, IC4 4081D, IC5 MICRF010, IC6 ADP2302, Q1 BSS84, Q3 13.4916mhz

Commit message: updated sch files
Parts:
- removed Q2: (no value), dp_devices:TRANSISTOR_FET_TSM2301CX
- removed R6: 50k, adafruit:R-US_R1206
- removed R8: 100k, adafruit:R-US_R1206
- removed R9: 100, adafruit:R-US_R1206
- added F1: PTCSMD, sparkfun:PTCSMD
- added JP10, JP9: M01, sparkfun:M01-SMTSO-256-ET
- added JP6, JP8: (no value), sparkfun:M03PTH
- added S3: REED-SWITCH, switch-reed:REED-SWITCH-CT10-1530-G1
- R5: value 50k -> 1k
Connections:
- removed net LED_ON: IC2.PD4(XCK/T0), R9.1
- removed net N$16: C1.1, IC6.EN, IC6.VIN, Q1.S, R10.2, R5.2, U$1.C
- removed net SHUT: IC5.SHUT, R8.2
- removed net VOLT: IC2.AREF, R5.1, R6.2
- new net A6: IC2.ADC6, JP6.3
- new net A7: IC2.ADC7, JP8.3
- new net REED: IC2.PD2(INT0), R5.1, S3.2
- net AGND: no longer R8.1
- net GND: now also JP1.2, JP10.1, JP2.2, JP3.2, JP4.2, JP6.1, JP8.1, S3.1; no longer Q2.S, R6.1
- net MOSI0: now also JP1.3; no longer JP1.4
- net MOSI1: now also JP2.3; no longer JP2.4
- net MOSI2: now also JP3.3; no longer JP3.4
- net MOSI3: now also JP4.3; no longer JP4.4
- net N$15: now also F1.1, JP9.1; no longer Q2.G, R9.2
- net N$8: now also C1.1, IC6.EN, IC6.VIN, Q1.S, R10.2, U$1.C; no longer JP1.2, JP2.2, JP3.2, JP4.2, Q2.D
- net SCK0: now also JP1.4; no longer JP1.3
- net SCK1: now also JP2.4; no longer JP2.3
- net SCK2: now also JP3.4; no longer JP3.3
- net SCK3: now also JP4.4; no longer JP4.3
- net VCC: now also F1.2, IC5.SHUT, JP6.2, JP8.2, R5.2
Other:
- note added: "Analog Breakout"
- note added: "Magnetic Detector"
- moved on the sheet: IC3A, IC3B, IC3C, IC3D, IC3P, IC4A, IC4B, IC4C, IC4D, IC4P, JP1, JP2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
