File: led_remote.sch (EAGLE design)
At the start: 26 parts, among them IC1 MICRF113, IC2 MEGA8-AI, Q1 13.56mhz

Commit message: updated sch files
Other:
- moved on the sheet: PCB2
Changed lines of the file:
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@@
 <instance part="P+6" gate="1" x="45.72" y="149.86" rot="R270"/>
 <instance part="GND7" gate="1" x="45.72" y="132.08" rot="R90"/>
-<instance part="PCB2" gate="G$1" x="127" y="40.64"/>
+<instance part="PCB2" gate="G$1" x="91.44" y="35.56"/>
 </instances>
 <busses>
